Commit message: Added models for the mecabot X
Used for the dimensions of the robot

File: src/wheeltec_ros2/src/transbot/core/wheeltec_robot_urdf/urdf/dongguan.urdf (robot description, URDF)
Before this commit: robot dongguan, 5 links, 4 joints
Links:
- link left_front_link: geometry visual cylinder length=0.05 radius=0.1
- link left_wheel_link: geometry visual cylinder length=0.05 radius=0.1
- link right_front_link: geometry visual cylinder length=0.05 radius=0.01
- link right_wheel_link: geometry visual cylinder length=0.05 radius=0.1
Joints:
- joint left_front_joint: origin xyz=0.175 0.28 0.075 rpy=1.57 0 0 -> xyz=0.214 0.247 0.1 rpy=1.57 0 0
- joint left_wheel_joint: origin xyz=-0.175 0.28 0.075 rpy=1.57 0 0 -> xyz=-0.214 0.47 0.1 rpy=1.57 0 0
- joint right_front_joint: origin xyz=0.175 -0.28 0.075 rpy=1.57 0 0 -> xyz=0.214 -0.247 0.1 rpy=1.57 0 0
- joint right_wheel_joint: origin xyz=-0.175 -0.28 0.075 rpy=1.57 0 0 -> xyz=-0.214 -0.247 0.1 rpy=1.57 0 0

Commit message: Fixed typo in .urdf file for Mecabot X

File: src/wheeltec_ros2/src/transbot/core/wheeltec_robot_urdf/urdf/dongguan.urdf (robot description, URDF)
Before this commit: robot dongguan, 5 links, 4 joints
Links:
- link right_front_link: geometry visual cylinder length=0.05 radius=0.1
Joints:
- joint left_wheel_joint: origin xyz=-0.214 0.47 0.1 rpy=1.57 0 0 -> xyz=-0.214 0.247 0.1 rpy=1.57 0 0
